File: pcb/rev1/Encoder.sch (KiCad schematic (older format))
At the start: 15 parts, among them P10 Port_Encoder, U11 iC-PV, U12 iC-MHM, U13 24LC16B

Commit message: updated schematics and added split PCB.
Parts:
- C55, C56, C57, C58, C59, C60: symbol Device:C_Small -> Motor_Gen2-rescue:C_Small-Device
- P10: symbol Connector_Generic:Conn_01x06 -> Motor_Gen2-rescue:Conn_01x06-Connector_Generic
- R27, R28, R29, R30, R31: symbol Device:R_Small -> Motor_Gen2-rescue:R_Small-Device
- U11: symbol RoMeLa_Motor:iC-PV -> Motor_Gen2-rescue:iC-PV-RoMeLa_Motor
- U12: symbol RoMeLa_Motor:iC-MHM -> Motor_Gen2-rescue:iC-MHM-RoMeLa_Motor
- U13: symbol RoMeLa_Motor:24LC16B -> Motor_Gen2-rescue:24LC16B-RoMeLa_Motor
Changed lines of the file:
@@
 encoding utf-8
 Sheet 6 7
-Title ""
-Date ""
-Rev ""
-Comp ""
-Comment1 ""
+Title "RoMeLa Motor Gen2"
+Date "2020-04-20"
+Rev "1.0"
+Comp "Robotics & Mechanisms Labratory(RoMeLa) UCLA"
+Comment1 "Author: Tym Zhu"
 Comment2 ""
 Comment3 ""
@@
 MOSI
 $Comp
-L Device:C_Small C55
+L Motor_Gen2-rescue:C_Small-Device C55
 U 1 1 5829923F
 P 6500 2250
@@
 $EndComp
 $Comp
-L power:GND #PWR0102
+L Motor_Gen2-rescue:GND-power #PWR0102
 U 1 1 582992A6
 P 6250 4350
@@
 $EndComp
 $Comp
-L power:GND #PWR093
+L Motor_Gen2-rescue:GND-power #PWR093
 U 1 1 5829936E
 P 6500 2450
@@
 $EndComp
 $Comp
-L RoMeLa_Motor:iC-MHM U12
+L Motor_Gen2-rescue:iC-MHM-RoMeLa_Motor U12
 U 1 1 5E212B3D
 P 6350 3400
@@
 	6250 2150 6250 2600
 $Comp
-L RoMeLa_Motor:iC-PV U11
+L Motor_Gen2-rescue:iC-PV-RoMeLa_Motor U11
 U 1 1 5E222BD8
 P 3250 3400
@@
 $EndComp
 $Comp
-L power:GND #PWR098
+L Motor_Gen2-rescue:GND-power #PWR098
 U 1 1 5E2237BA
 P 2200 3500
@@
 	3900 3650 5600 3650
 $Comp
-L Device:R_Small R30
+L Motor_Gen2-rescue:R_Small-Device R30
 U 1 1 5E2366C8
 P 2000 3400
@@
 $EndComp
 $Comp
-L power:GND #PWR097
+L Motor_Gen2-rescue:GND-power #PWR097
 U 1 1 5E2378C8
 P 2000 3500
@@
 $EndComp
 $Comp
-L Device:R_Small R31
+L Motor_Gen2-rescue:R_Small-Device R31
 U 1 1 5E237A97
 P 2300 3900
@@
 	2300 3700 2300 3800
 $Comp
-L power:GND #PWR0100
+L Motor_Gen2-rescue:GND-power #PWR0100
 U 1 1 5E23868B
 P 2300 4000
@@
 	2500 3300 2000 3300
 $Comp
-L power:GND #PWR0101
+L Motor_Gen2-rescue:GND-power #PWR0101
 U 1 1 5E23CF72
 P 3300 4250
@@
 $EndComp
 $Comp
-L power:GND #PWR094
+L Motor_Gen2-rescue:GND-power #PWR094
 U 1 1 5E23DD79
 P 2350 2550
@@
 BATT-
 $Comp
-L Device:R_Small R27
+L Motor_Gen2-rescue:R_Small-Device R27
 U 1 1 5E23F0AC
 P 1700 2250
@@
 $EndComp
 $Comp
-L Device:R_Small R28
+L Motor_Gen2-rescue:R_Small-Device R28
 U 1 1 5E23FA6C
 P 2050 2250
@@
 	2350 2300 2350 2250
 $Comp
-L Device:C_Small C58
+L Motor_Gen2-rescue:C_Small-Device C58
 U 1 1 5E23D3B5
 P 2350 2400
@@
 Connection ~ 2350 2500
 $Comp
-L Device:C_Small C59
+L Motor_Gen2-rescue:C_Small-Device C59
 U 1 1 5E2434B9
 P 4300 2950
@@
 	3900 2850 4300 2850
 $Comp
-L power:GND #PWR095
+L Motor_Gen2-rescue:GND-power #PWR095
 U 1 1 5E244431
 P 4300 3050
@@
 SDA
 $Comp
-L RoMeLa_Motor:24LC16B U13
+L Motor_Gen2-rescue:24LC16B-RoMeLa_Motor U13
 U 1 1 5E24A47C
 P 4650 5200
@@
 SDA
 $Comp
-L power:GND #PWR0106
+L Motor_Gen2-rescue:GND-power #PWR0106
 U 1 1 5E24AFD9
 P 4650 5500
@@
 $EndComp
 $Comp
-L power:GND #PWR0105
+L Motor_Gen2-rescue:GND-power #PWR0105
 U 1 1 5E24B421
 P 5050 5300
@@
 $EndComp
 $Comp
-L Device:C_Small C60
+L Motor_Gen2-rescue:C_Small-Device C60
 U 1 1 5E24B84A
 P 4850 4650
@@
 $EndComp
 $Comp
-L power:GND #PWR0104
+L Motor_Gen2-rescue:GND-power #PWR0104
 U 1 1 5E24D041
 P 4850 4750
@@
 	4650 4550 4650 4900
 $Comp
-L power:+5V #PWR089
+L Motor_Gen2-rescue:+5V-power #PWR089
 U 1 1 5E25A4C9
 P 6250 2100
@@
 $EndComp
 $Comp
-L power:+5V #PWR091
+L Motor_Gen2-rescue:+5V-power #PWR091
 U 1 1 5E25AF4D
 P 3400 2200
@@
 	3400 2200 3400 2250
 $Comp
-L Device:C_Small C56
+L Motor_Gen2-rescue:C_Small-Device C56
 U 1 1 5E25CD59
 P 6850 2250
@@
 	6500 2400 6500 2350
 $Comp
-L Device:R_Small R29
+L Motor_Gen2-rescue:R_Small-Device R29
 U 1 1 5E25FD27
 P 5400 3050
@@
 	5500 3050 5600 3050
 $Comp
-L power:+5V #PWR0103
+L Motor_Gen2-rescue:+5V-power #PWR0103
 U 1 1 5E267BCA
 P 4650 4500
@@
 NoConn ~ 7000 3100
 $Comp
-L Device:C_Small C57
+L Motor_Gen2-rescue:C_Small-Device C57
 U 1 1 5E26D51A
 P 3650 2350
@@
 $EndComp
 $Comp
-L power:GND #PWR092
+L Motor_Gen2-rescue:GND-power #PWR092
 U 1 1 5E26D9E7
 P 3650 2450
@@
 SCLK
 $Comp
-L Connector_Generic:Conn_01x06 P?
+L Motor_Gen2-rescue:Conn_01x06-Connector_Generic P?
 U 1 1 5E99C8B7
 P 9150 3600
@@
 $EndComp
 $Comp
-L power:GND #PWR?
+L Motor_Gen2-rescue:GND-power #PWR?
 U 1 1 5E99C8BD
 P 8450 3600
@@
 Connection ~ 2350 2250
 $Comp
-L power:+5V #PWR0121
+L Motor_Gen2-rescue:+5V-power #PWR0121
 U 1 1 5E2BEDC3
 P 8750 3300
