File: pcb/rev1/Motor_Gen2.sch (KiCad schematic (older format))
At the start: 17 parts, among them J1 PicoBlade 6P, J2 PicoBlade 6P, P1 +IN, P11 -IN, P2 MT_A, P3 MT_B, P4 MT_C, P5 CONN_BATT, P6 CONN_TC

Commit message: updated schematics and added split PCB.
Parts:
- BT1: symbol Device:Battery_Cell -> Motor_Gen2-rescue:Battery_Cell-Device
- C26: symbol Device:C_Small -> Motor_Gen2-rescue:C_Small-Device
- H1, H2, H3, H4: symbol Mechanical:MountingHole_Pad -> Motor_Gen2-rescue:MountingHole_Pad-Mechanical
- J1, J2: symbol Connector_Generic:Conn_01x06 -> Motor_Gen2-rescue:Conn_01x06-Connector_Generic
- P1, P11, P2, P3, P4: symbol Connector:TestPoint -> Motor_Gen2-rescue:TestPoint-Connector
- P5, P6: symbol Connector_Generic:Conn_01x02 -> Motor_Gen2-rescue:Conn_01x02-Connector_Generic
- R1: symbol Device:R_Small -> Motor_Gen2-rescue:R_Small-Device
- R38: symbol Device:R -> Motor_Gen2-rescue:R-Device
Changed lines of the file:
@@
 $EndSheet
 $Comp
-L Device:R_Small R1
+L Motor_Gen2-rescue:R_Small-Device R1
 U 1 1 58299209
 P 2400 1650
@@
 $EndComp
 $Comp
-L power:GNDREF #PWR03
+L Motor_Gen2-rescue:GNDREF-power #PWR03
 U 1 1 5829962A
 P 2600 1650
@@
 $EndComp
 $Comp
-L Connector_Generic:Conn_01x02 P6
+L Motor_Gen2-rescue:Conn_01x02-Connector_Generic P6
 U 1 1 582AC713
 P 2100 4300
@@
 $EndComp
 $Comp
-L Connector:TestPoint P2
+L Motor_Gen2-rescue:TestPoint-Connector P2
 U 1 1 582AB0F8
 P 7900 2150
@@
 $EndComp
 $Comp
-L Connector:TestPoint P3
+L Motor_Gen2-rescue:TestPoint-Connector P3
 U 1 1 582ABC63
 P 7900 2350
@@
 $EndComp
 $Comp
-L Connector:TestPoint P4
+L Motor_Gen2-rescue:TestPoint-Connector P4
 U 1 1 582ABE29
 P 7900 2550
@@
 	3950 4100 4450 4100
 $Comp
-L power:+48V #PWR01
+L Motor_Gen2-rescue:+48V-power #PWR01
 U 1 1 5832C1E8
 P 8900 1450
@@
 	8100 4450 7900 4450
 $Comp
-L power:GNDPWR #PWR02
+L Motor_Gen2-rescue:GNDPWR-power #PWR02
 U 1 1 5832E244
 P 8900 1550
@@
 	3950 2200 4450 2200
 $Comp
-L Connector_Generic:Conn_01x06 J2
+L Motor_Gen2-rescue:Conn_01x06-Connector_Generic J2
 U 1 1 5EA13651
 P 1450 2550
@@
 $EndComp
 $Comp
-L Connector_Generic:Conn_01x06 J1
+L Motor_Gen2-rescue:Conn_01x06-Connector_Generic J1
 U 1 1 5EA1E3F2
 P 1450 1850
@@
 Connection ~ 2150 2450
 $Comp
-L Device:Battery_Cell BT1
+L Motor_Gen2-rescue:Battery_Cell-Device BT1
 U 1 1 5EA51518
 P 2250 3450
@@
 $EndComp
 $Comp
-L Connector_Generic:Conn_01x02 P5
+L Motor_Gen2-rescue:Conn_01x02-Connector_Generic P5
 U 1 1 5EA52F07
 P 1450 3550
@@
 Connection ~ 2250 3250
 $Comp
-L power:GNDPWR #PWR0113
+L Motor_Gen2-rescue:GNDPWR-power #PWR0113
 U 1 1 5E0E9B26
 P 2050 6300
@@
 $EndComp
 $Comp
-L Mechanical:MountingHole_Pad H1
+L Motor_Gen2-rescue:MountingHole_Pad-Mechanical H1
 U 1 1 5E0FA87A
 P 2050 5600
@@
 $EndComp
 $Comp
-L Connector:TestPoint P1
+L Motor_Gen2-rescue:TestPoint-Connector P1
 U 1 1 5E2D6D9C
 P 8900 1450
@@
 $EndComp
 $Comp
-L Connector:TestPoint P11
+L Motor_Gen2-rescue:TestPoint-Connector P11
 U 1 1 5E2D7645
 P 8900 1550
@@
 $EndComp
 $Comp
-L Mechanical:MountingHole_Pad H2
+L Motor_Gen2-rescue:MountingHole_Pad-Mechanical H2
 U 1 1 5E2E12CF
 P 2350 5600
@@
 $EndComp
 $Comp
-L Mechanical:MountingHole_Pad H3
+L Motor_Gen2-rescue:MountingHole_Pad-Mechanical H3
 U 1 1 5E2E15B2
 P 2650 5600
@@
 $EndComp
 $Comp
-L Mechanical:MountingHole_Pad H4
+L Motor_Gen2-rescue:MountingHole_Pad-Mechanical H4
 U 1 1 5E2E1805
 P 2950 5600
@@
 Connection ~ 2350 5700
 $Comp
-L Device:C_Small C?
+L Motor_Gen2-rescue:C_Small-Device C?
 U 1 1 5E2FC9E6
 P 2050 6000
@@
 C0805W472KDRACTU
 $Comp
-L power:Earth_Protective #PWR0118
+L Motor_Gen2-rescue:Earth_Protective-power #PWR0118
 U 1 1 5E1D66A0
 P 2950 5700
@@
 Connection ~ 2050 5700
 $Comp
-L Device:R R38
+L Motor_Gen2-rescue:R-Device R38
 U 1 1 5E1EE096
 P 1700 6000
@@
 	2050 6100 2050 6250
 $Comp
-L power:+BATT #PWR0119
+L Motor_Gen2-rescue:+BATT-power #PWR0119
 U 1 1 5E22C2C9
 P 2250 3250
