File: pcb/split/gen2L/RS485.sch (KiCad schematic (older format))
At the start: 14 parts, among them U14 ISOW7842F, U15 MAX14775E

Commit message: updated schematics and added split PCB.
Parts:
- C61, C62, C63, C64, C65: symbol Motor_Gen2-rescue:C_Small-Device -> Motor_Gen2L-rescue:C_Small-Device
- D5: symbol Motor_Gen2-rescue:D_TVS_x2_AAC-Device -> Motor_Gen2L-rescue:D_TVS_x2_AAC-Device
- D6: symbol Motor_Gen2-rescue:D_ALT-Device -> Motor_Gen2L-rescue:D_ALT-Device
- F1: symbol Motor_Gen2-rescue:Polyfuse-Device -> Motor_Gen2L-rescue:Polyfuse-Device
- R32, R33, R34, R35: symbol Motor_Gen2-rescue:R_Small-Device -> Motor_Gen2L-rescue:R_Small-Device
- U15: symbol Motor_Gen2-rescue:MAX14775E-RoMeLa_Motor -> Motor_Gen2L-rescue:MAX14775E-RoMeLa_Motor
Connections:
- net A: now also D5.1 (A1); no longer D5.2 (A2)
- net B: now also D5.2 (A2); no longer D5.1 (A1)
Changed lines of the file:
@@
 $Descr A4 11693 8268
 encoding utf-8
-Sheet 7 7
-Title "RoMeLa Motor Gen2"
-Date "2020-04-20"
+Sheet 5 5
+Title "RoMeLa Motor Gen2 Logic Board"
+Date "10/27/2022"
 Rev "1.0"
 Comp "Robotics & Mechanisms Labratory(RoMeLa) UCLA"
@@
 $EndDescr
 $Comp
-L Motor_Gen2-rescue:GNDREF-power #PWR0109
+L Motor_Gen2L-rescue:GNDREF-power #PWR0109
 U 1 1 582AD43A
 P 5400 2650
@@
 TxD
 $Comp
-L Motor_Gen2-rescue:C_Small-Device C61
+L Motor_Gen2L-rescue:C_Small-Device C61
 U 1 1 582AD5E4
 P 3600 2500
@@
 $EndComp
 $Comp
-L Motor_Gen2-rescue:C_Small-Device C62
+L Motor_Gen2L-rescue:C_Small-Device C62
 U 1 1 582AD5EA
 P 3800 2500
@@
 $EndComp
 $Comp
-L Motor_Gen2-rescue:GND-power #PWR0108
+L Motor_Gen2L-rescue:GND-power #PWR0108
 U 1 1 582AD5F5
 P 3600 2650
@@
 $EndComp
 $Comp
-L Motor_Gen2-rescue:C_Small-Device C64
+L Motor_Gen2L-rescue:C_Small-Device C64
 U 1 1 582AD7B1
 P 5400 2500
@@
 $EndComp
 $Comp
-L Motor_Gen2-rescue:C_Small-Device C63
+L Motor_Gen2L-rescue:C_Small-Device C63
 U 1 1 582AD7B7
 P 5200 2500
@@
 $EndComp
 $Comp
-L Motor_Gen2-rescue:C_Small-Device C65
+L Motor_Gen2L-rescue:C_Small-Device C65
 U 1 1 582AD967
 P 6000 2500
@@
 B
 $Comp
-L Motor_Gen2-rescue:R_Small-Device R32
+L Motor_Gen2L-rescue:R_Small-Device R32
 U 1 1 58297025
 P 7150 2850
@@
 $EndComp
 $Comp
-L Motor_Gen2-rescue:R_Small-Device R33
+L Motor_Gen2L-rescue:R_Small-Device R33
 U 1 1 58297159
 P 7150 3150
@@
 $EndComp
 $Comp
-L Motor_Gen2-rescue:+3.3V-power #PWR0107
+L Motor_Gen2L-rescue:+3.3V-power #PWR0107
 U 1 1 582C8BD5
 P 3600 2350
@@
 	6100 2850 5850 2850
 $Comp
-L Motor_Gen2-rescue:GNDREF-power #PWR0110
+L Motor_Gen2L-rescue:GNDREF-power #PWR0110
 U 1 1 5E2BB050
 P 6500 3550
@@
 	4950 3150 6100 3150
 $Comp
-L Motor_Gen2-rescue:MAX14775E-RoMeLa_Motor U15
+L Motor_Gen2L-rescue:MAX14775E-RoMeLa_Motor U15
 U 1 1 5E2B407C
 P 6500 2950
@@
 3.3Viso
 $Comp
-L Motor_Gen2-rescue:R_Small-Device R34
+L Motor_Gen2L-rescue:R_Small-Device R34
 U 1 1 5E2DB91D
 P 5950 4000
@@
 Connection ~ 5950 4200
 $Comp
-L Motor_Gen2-rescue:GNDREF-power #PWR0112
+L Motor_Gen2L-rescue:GNDREF-power #PWR0112
 U 1 1 5E2E91C9
 P 5950 4650
@@
 $EndComp
 $Comp
-L Motor_Gen2-rescue:D_ALT-Device D6
+L Motor_Gen2L-rescue:D_ALT-Device D6
 U 1 1 5E2EAFDD
 P 5950 4500
@@
 ISO_DI
 $Comp
-L Motor_Gen2-rescue:R_Small-Device R35
+L Motor_Gen2L-rescue:R_Small-Device R35
 U 1 1 5E2F3594
 P 5350 4200
@@
 	6600 4200 5950 4200
 $Comp
-L Motor_Gen2-rescue:Polyfuse-Device F1
+L Motor_Gen2L-rescue:Polyfuse-Device F1
 U 1 1 5E2F87B2
 P 6750 4200
@@
 SMF3.3
 $Comp
-L Motor_Gen2-rescue:D_TVS_x2_AAC-Device D5
+L Motor_Gen2L-rescue:D_TVS_x2_AAC-Device D5
 U 1 1 5E30313B
 P 7700 3600
@@
 F 3 "~" H 7550 3600 50  0001 C CNN
 	1    7700 3600
-	1    0    0    -1
-$EndComp
-$Comp
-L Motor_Gen2-rescue:GNDREF-power #PWR0111
+	-1   0    0    -1
+$EndComp
+$Comp
+L Motor_Gen2L-rescue:GNDREF-power #PWR0111
 U 1 1 5E30A298
 P 7700 3750
