File: pcb/split/gen2L/stm32.sch (KiCad schematic (older format))
At the start: 21 parts, among them P7 Port_SW, P8 CONN_01X04, P9 Port_Encoder, U1 446, Y1 Resonator

Commit message: updated schematics and added split PCB.
Parts:
- added C16: 104, Capacitor_SMD:C_0402_1005Metric, symbol Motor_Gen2L-rescue:C_Small-Device
- added R25, R26: 3.9k, Resistor_SMD:R_0402_1005Metric, symbol Motor_Gen2L-rescue:R_Small-Device
- C1, C2, C3, C4, C5, C6, C7: symbol Motor_Gen2-rescue:C_Small-Device -> Motor_Gen2L-rescue:C_Small-Device
- D1, D2, D3: symbol Motor_Gen2-rescue:LED-Device -> Motor_Gen2L-rescue:LED-Device
- JP1, JP2: symbol Motor_Gen2-rescue:SolderJumper_2_Open-Jumper -> Motor_Gen2L-rescue:SolderJumper_2_Open-Jumper
- P7: symbol Motor_Gen2-rescue:Conn_01x06-Connector_Generic -> Motor_Gen2L-rescue:Conn_01x06-Connector_Generic
- P8: symbol Motor_Gen2-rescue:Conn_01x04-Connector_Generic -> Motor_Gen2L-rescue:Conn_01x04-Connector_Generic
- P9: footprint RoMeLa_Motor:FFC_8POS_0.5mm_TOP -> RoMeLa_Motor:FFC_8POS_0.5mm_BackFlip; symbol Motor_Gen2-rescue:Conn_01x08-Connector_Generic -> Motor_Gen2L-rescue:Conn_01x08-Connector_Generic
- R2: symbol Motor_Gen2-rescue:R_Small-Device -> Motor_Gen2L-rescue:R_Small-Device
- R3, R4, R5: symbol Motor_Gen2-rescue:R-Device -> Motor_Gen2L-rescue:R-Device
- U1: symbol Motor_Gen2-rescue:446-RoMeLa_Motor -> Motor_Gen2L-rescue:446-RoMeLa_Motor
- Y1: symbol Motor_Gen2-rescue:Resonator-Device -> Motor_Gen2L-rescue:Resonator-Device
Connections:
- net +3V3: now also R25.1, R26.1
- net GND: now also C16.2
- net I2C_SCL: now also R26.2
- net I2C_SDA: now also R25.2
- net PVDDSENSE: now also C16.1
Changed lines of the file:
@@
 $Descr A4 11693 8268
 encoding utf-8
-Sheet 2 7
-Title "RoMeLa Motor Gen2"
-Date "2020-04-20"
+Sheet 2 5
+Title "RoMeLa Motor Gen2 Logic Board"
+Date "10/27/2022"
 Rev "1.0"
 Comp "Robotics & Mechanisms Labratory(RoMeLa) UCLA"
@@
 Text HLabel 2700 2200 0    60   Input ~ 0
 FAULT
-Text HLabel 2700 2600 0    60   Input ~ 0
+Text HLabel 1850 2600 0    60   Input ~ 0
 PVDDSENSE
 Text HLabel 2700 3900 0    60   Input ~ 0
@@
 485_TX
 $Comp
-L Motor_Gen2-rescue:446-RoMeLa_Motor U1
+L Motor_Gen2L-rescue:446-RoMeLa_Motor U1
 U 1 1 582C559B
 P 2700 1000
@@
 $EndComp
 $Comp
-L Motor_Gen2-rescue:446-RoMeLa_Motor U1
+L Motor_Gen2L-rescue:446-RoMeLa_Motor U1
 U 2 1 582C55B2
 P 2700 2600
@@
 $EndComp
 $Comp
-L Motor_Gen2-rescue:446-RoMeLa_Motor U1
+L Motor_Gen2L-rescue:446-RoMeLa_Motor U1
 U 3 1 582C55CB
 P 2700 4300
@@
 $EndComp
 $Comp
-L Motor_Gen2-rescue:446-RoMeLa_Motor U1
+L Motor_Gen2L-rescue:446-RoMeLa_Motor U1
 U 4 1 582C55E6
 P 2700 5900
@@
 $EndComp
 $Comp
-L Motor_Gen2-rescue:446-RoMeLa_Motor U1
+L Motor_Gen2L-rescue:446-RoMeLa_Motor U1
 U 5 1 582C561A
 P 5650 3050
@@
 $EndComp
 $Comp
-L Motor_Gen2-rescue:446-RoMeLa_Motor U1
+L Motor_Gen2L-rescue:446-RoMeLa_Motor U1
 U 6 1 582C564F
 P 5600 1100
@@
 Text HLabel 1900 5300 0    60   Input ~ 0
 TC_SO
-Text HLabel 2700 3500 0    60   BiDi ~ 0
+Text HLabel 1100 3500 0    60   BiDi ~ 0
 I2C_SDA
-Text HLabel 2700 3400 0    60   Output ~ 0
+Text HLabel 1100 3400 0    60   Output ~ 0
 I2C_SCL
 $Comp
-L Motor_Gen2-rescue:+3.3V-power #PWR04
+L Motor_Gen2L-rescue:+3.3V-power #PWR04
 U 1 1 582C8FBD
 P 5500 1000
@@
 Connection ~ 5500 1600
 $Comp
-L Motor_Gen2-rescue:GND-power #PWR08
+L Motor_Gen2L-rescue:GND-power #PWR08
 U 1 1 582C90AB
 P 5500 2300
@@
 Connection ~ 5500 2200
 $Comp
-L Motor_Gen2-rescue:C_Small-Device C6
+L Motor_Gen2L-rescue:C_Small-Device C6
 U 1 1 582C9189
 P 5050 1350
@@
 $EndComp
 $Comp
-L Motor_Gen2-rescue:GND-power #PWR07
+L Motor_Gen2L-rescue:GND-power #PWR07
 U 1 1 582C91C6
 P 5050 1450
@@
 NRST
 $Comp
-L Motor_Gen2-rescue:R_Small-Device R2
+L Motor_Gen2L-rescue:R_Small-Device R2
 U 1 1 582C93A1
 P 5000 3050
@@
 	5100 3050 5650 3050
 $Comp
-L Motor_Gen2-rescue:GND-power #PWR011
+L Motor_Gen2L-rescue:GND-power #PWR011
 U 1 1 582C9419
 P 4700 3200
@@
 	4700 3050 4900 3050
 $Comp
-L Motor_Gen2-rescue:C_Small-Device C7
+L Motor_Gen2L-rescue:C_Small-Device C7
 U 1 1 582C950B
 P 5000 3350
@@
 	5000 3150 5650 3150
 $Comp
-L Motor_Gen2-rescue:GND-power #PWR012
+L Motor_Gen2L-rescue:GND-power #PWR012
 U 1 1 582C9573
 P 5000 3450
@@
 NoConn ~ 5650 3550
 $Comp
-L Motor_Gen2-rescue:Resonator-Device Y1
+L Motor_Gen2L-rescue:Resonator-Device Y1
 U 1 1 582C9864
 P 5350 4100
@@
 $EndComp
 $Comp
-L Motor_Gen2-rescue:GND-power #PWR015
+L Motor_Gen2L-rescue:GND-power #PWR015
 U 1 1 582C98AF
 P 5350 4300
@@
 	5600 3750 5600 4100
 $Comp
-L Motor_Gen2-rescue:C_Small-Device C1
+L Motor_Gen2L-rescue:C_Small-Device C1
 U 1 1 582C99AD
 P 6800 1300
@@
 $EndComp
 $Comp
-L Motor_Gen2-rescue:C_Small-Device C2
+L Motor_Gen2L-rescue:C_Small-Device C2
 U 1 1 582C99E7
 P 7000 1300
@@
 $EndComp
 $Comp
-L Motor_Gen2-rescue:C_Small-Device C3
+L Motor_Gen2L-rescue:C_Small-Device C3
 U 1 1 582C9A1A
 P 7200 1300
@@
 $EndComp
 $Comp
-L Motor_Gen2-rescue:C_Small-Device C4
+L Motor_Gen2L-rescue:C_Small-Device C4
 U 1 1 582C9A52
 P 7400 1300
@@
 $EndComp
 $Comp
-L Motor_Gen2-rescue:C_Small-Device C5
+L Motor_Gen2L-rescue:C_Small-Device C5
 U 1 1 582C9A8B
 P 7600 1300
@@
 Connection ~ 7400 1400
 $Comp
-L Motor_Gen2-rescue:GND-power #PWR06
+L Motor_Gen2L-rescue:GND-power #PWR06
 U 1 1 582C9D10
 P 6800 1400
@@
 Connection ~ 6800 1200
 $Comp
-L Motor_Gen2-rescue:+3.3V-power #PWR05
+L Motor_Gen2L-rescue:+3.3V-power #PWR05
 U 1 1 582C9D4C
 P 6800 1200
@@
 $EndComp
 $Comp
-L Motor_Gen2-rescue:Conn_01x06-Connector_Generic P7
+L Motor_Gen2L-rescue:Conn_01x06-Connector_Generic P7
 U 1 1 582C9E0D
 P 9400 3100
@@
 $EndComp
 $Comp
-L Motor_Gen2-rescue:+3.3V-power #PWR09
+L Motor_Gen2L-rescue:+3.3V-power #PWR09
 U 1 1 582C9E5E
 P 9000 2800
@@
 SWCLK
 $Comp
-L Motor_Gen2-rescue:GND-power #PWR010
+L Motor_Gen2L-rescue:GND-power #PWR010
 U 1 1 582C9F14
 P 8600 3100
@@
 DEBUG
 $Comp
-L Motor_Gen2-rescue:Conn_01x04-Connector_Generic P8
+L Motor_Gen2L-rescue:Conn_01x04-Connector_Generic P8
 U 1 1 582CA665
 P 9400 3950
@@
 $EndComp
 $Comp
-L Motor_Gen2-rescue:GND-power #PWR014
+L Motor_Gen2L-rescue:GND-power #PWR014
 U 1 1 582CA6AC
 P 9200 4150
@@
 $EndComp
 $Comp
-L Motor_Gen2-rescue:+3.3V-power #PWR013
+L Motor_Gen2L-rescue:+3.3V-power #PWR013
 U 1 1 582CA96D
 P 9000 3750
@@
 LED_B
 $Comp
-L Motor_Gen2-rescue:LED-Device D1
+L Motor_Gen2L-rescue:LED-Device D1
 U 1 1 5831BFC7
 P 5600 5500
@@
 $EndComp
 $Comp
-L Motor_Gen2-rescue:LED-Device D2
+L Motor_Gen2L-rescue:LED-Device D2
 U 1 1 5831C132
 P 6000 5500
@@
 $EndComp
 $Comp
-L Motor_Gen2-rescue:LED-Device D3
+L Motor_Gen2L-rescue:LED-Device D3
 U 1 1 5831C187
 P 6400 5500
@@
 $EndComp
 $Comp
-L Motor_Gen2-rescue:R-Device R3
+L Motor_Gen2L-rescue:R-Device R3
 U 1 1 5831C893
 P 5600 5200
@@
 $EndComp
 $Comp
-L Motor_Gen2-rescue:R-Device R4
+L Motor_Gen2L-rescue:R-Device R4
 U 1 1 5831C975
 P 6000 5200
@@
 $EndComp
 $Comp
-L Motor_Gen2-rescue:R-Device R5
+L Motor_Gen2L-rescue:R-Device R5
 U 1 1 5831CA15
 P 6400 5200
@@
 LED_B
 $Comp
-L Motor_Gen2-rescue:GND-power #PWR018
+L Motor_Gen2L-rescue:GND-power #PWR018
 U 1 1 5831D7F2
 P 5600 5650
@@
 $EndComp
 $Comp
-L Motor_Gen2-rescue:GND-power #PWR019
+L Motor_Gen2L-rescue:GND-power #PWR019
 U 1 1 5831D842
 P 6000 5650
@@
 $EndComp
 $Comp
-L Motor_Gen2-rescue:GND-power #PWR020
+L Motor_Gen2L-rescue:GND-power #PWR020
 U 1 1 5831D892
 P 6400 5650
@@
 	2250 3600 2700 3600
 $Comp
-L Motor_Gen2-rescue:Conn_01x08-Connector_Generic P9
+L Motor_Gen2L-rescue:Conn_01x08-Connector_Generic P9
 U 1 1 590D4639
 P 9400 5400
 F 0 "P9" H 9400 5800 50  0000 C CNN
 F 1 "Port_Encoder" V 9500 5400 50  0000 C CNN
-F 2 "RoMeLa_Motor:FFC_8POS_0.5mm_TOP" H 9400 5400 50  0001 C CNN
+F 2 "RoMeLa_Motor:FFC_8POS_0.5mm_BackFlip" H 9400 5400 50  0001 C CNN
 F 3 "" H 9400 5400 50  0000 C CNN
 	1    9400 5400
@@
 $EndComp
 $Comp
-L Motor_Gen2-rescue:GND-power #PWR017
+L Motor_Gen2L-rescue:GND-power #PWR017
 U 1 1 590D4CCD
 P 8500 5300
@@
 3.3V or 5V output!!!
 $Comp
-L Motor_Gen2-rescue:+5V-power #PWR0114
+L Motor_Gen2L-rescue:+5V-power #PWR0114
 U 1 1 5E111DC3
 P 9000 4700
@@
 $EndComp
 $Comp
-L Motor_Gen2-rescue:+3.3V-power #PWR0115
+L Motor_Gen2L-rescue:+3.3V-power #PWR0115
 U 1 1 5E1131C9
 P 8650 4700
@@
 Connection ~ 9000 5100
 $Comp
-L Motor_Gen2-rescue:SolderJumper_2_Open-Jumper JP1
+L Motor_Gen2L-rescue:SolderJumper_2_Open-Jumper JP1
 U 1 1 5E1F4226
 P 8650 4850
@@
 $EndComp
 $Comp
-L Motor_Gen2-rescue:SolderJumper_2_Open-Jumper JP2
+L Motor_Gen2L-rescue:SolderJumper_2_Open-Jumper JP2
 U 1 1 5E1F6784
 P 9000 4850
@@
 $EndComp
 $Comp
-L Motor_Gen2-rescue:+BATT-power #PWR0120
+L Motor_Gen2L-rescue:+BATT-power #PWR0120
 U 1 1 5E22DD47
 P 9200 5800
@@
 Text Label 9200 5700 2    60   ~ 0
 PRESET
-Text Label 1900 2700 2    60   ~ 0
+Text Label 2700 2700 2    60   ~ 0
 PRESET
-Wire Wire Line
-	1900 2700 2700 2700
 Text HLabel 2700 5200 0    60   Output ~ 0
 DRV_ENABLE
+Wire Wire Line
+	1850 2600 1900 2600
+$Comp
+L Motor_Gen2L-rescue:C_Small-Device C16
+U 1 1 63517695
+P 1900 2750
+F 0 "C16" H 1910 2820 50  0000 L CNN
+F 1 "104" H 1910 2670 50  0000 L CNN
+F 2 "Capacitor_SMD:C_0402_1005Metric" H 1900 2750 50  0001 C CNN
+F 3 "" H 1900 2750 50  0000 C CNN
+	1    1900 2750
+	1    0    0    -1
+$EndComp
+Wire Wire Line
+	1900 2650 1900 2600
+Connection ~ 1900 2600
+Wire Wire Line
+	1900 2600 2700 2600
+$Comp
+L Motor_Gen2L-rescue:GND-power #PWR0117
+U 1 1 635198D4
+P 1900 2850
+F 0 "#PWR0117" H 1900 2600 50  0001 C CNN
+F 1 "GND" H 1900 2700 50  0000 C CNN
+F 2 "" H 1900 2850 50  0000 C CNN
+F 3 "" H 1900 2850 50  0000 C CNN
+	1    1900 2850
+	1    0    0    -1
+$EndComp
+$Comp
+L Motor_Gen2L-rescue:R_Small-Device R26
+U 1 1 6350AD21
+P 1200 3250
+F 0 "R26" H 1250 3300 50  0000 L CNN
+F 1 "3.9k" H 1250 3200 50  0000 L CNN
+F 2 "Resistor_SMD:R_0402_1005Metric" H 1200 3250 50  0001 C CNN
+F 3 "" H 1200 3250 50  0000 C CNN
+	1    1200 3250
+	1    0    0    -1
+$EndComp
+Wire Wire Line
+	1100 3400 1200 3400
+Wire Wire Line
+	1200 3400 2700 3400
+Connection ~ 1200 3400
+Wire Wire Line
+	1200 3350 1200 3400
+$Comp
+L Motor_Gen2L-rescue:+3.3V-power #PWR0118
+U 1 1 6351148F
+P 1200 3150
+F 0 "#PWR0118" H 1200 3000 50  0001 C CNN
+F 1 "+3.3V" H 1200 3290 50  0000 C CNN
+F 2 "" H 1200 3150 50  0000 C CNN
+F 3 "" H 1200 3150 50  0000 C CNN
+	1    1200 3150
+	1    0    0    -1
+$EndComp
+$Comp
+L Motor_Gen2L-rescue:R_Small-Device R25
+U 1 1 63511D2D
+P 1500 3250
+F 0 "R25" H 1550 3300 50  0000 L CNN
+F 1 "3.9k" H 1550 3200 50  0000 L CNN
+F 2 "Resistor_SMD:R_0402_1005Metric" H 1500 3250 50  0001 C CNN
+F 3 "" H 1500 3250 50  0000 C CNN
+	1    1500 3250
+	1    0    0    -1
+$EndComp
+$Comp
+L Motor_Gen2L-rescue:+3.3V-power #PWR0122
+U 1 1 635123E6
+P 1500 3150
+F 0 "#PWR0122" H 1500 3000 50  0001 C CNN
+F 1 "+3.3V" H 1500 3290 50  0000 C CNN
+F 2 "" H 1500 3150 50  0000 C CNN
+F 3 "" H 1500 3150 50  0000 C CNN
+	1    1500 3150
+	1    0    0    -1
+$EndComp
+Wire Wire Line
+	1100 3500 1500 3500
+Wire Wire Line
+	1500 3350 1500 3500
+Connection ~ 1500 3500
+Wire Wire Line
+	1500 3500 2700 3500
 $EndSCHEMATC
