File: pcb/split/gen2P/Current_ADC.sch (KiCad schematic (older format))
At the start: 31 parts, among them U4 LP5912-5.0, U5 OPA2320, U6 INA240, U7 ADS8353, U8 INA240

Commit message: updated schematics and added split PCB.
Parts:
- removed C37: 104, Capacitor_SMD:C_0402_1005Metric, symbol Motor_Gen2-rescue:C_Small-Device
- removed C41, C45: 1.5nF C0G, Capacitor_SMD:C_0402_1005Metric, symbol Motor_Gen2-rescue:C_Small-Device
- removed C43, C46: 1nF C0G, Capacitor_SMD:C_0402_1005Metric, symbol Motor_Gen2-rescue:C_Small-Device
- removed R17, R21: 7.5k, Resistor_SMD:R_0402_1005Metric, symbol Motor_Gen2-rescue:R_Small-Device
- removed R18, R22: 13k, Resistor_SMD:R_0402_1005Metric, symbol Motor_Gen2-rescue:R_Small-Device
- removed U5: OPA2320, Package_SON:Texas_S-PWSON-N8_EP1.2x2mm, symbol Motor_Gen2-rescue:OPA2320-RoMeLa_Motor
- C33, C34, C35, C36, C38, C39, C40, C42, C48, C49: symbol Motor_Gen2-rescue:C_Small-Device -> Motor_Gen2P-rescue:C_Small-Device
- C44, C47: value 1.5nF C0G -> 1nF C0G; symbol Motor_Gen2-rescue:C_Small-Device -> Motor_Gen2P-rescue:C_Small-Device
- R16: footprint Resistor_SMD:R_0402_1005Metric -> NetTie:NetTie-2_SMD_Pad0.5mm; symbol Motor_Gen2-rescue:R_Small-Device -> Motor_Gen2P-rescue:R_Small-Device
- R19, R20, R23, R24: value 10 -> 33; symbol Motor_Gen2-rescue:R_Small-Device -> Motor_Gen2P-rescue:R_Small-Device
- U4: symbol Motor_Gen2-rescue:LP5912-5.0-RoMeLa_Motor -> Motor_Gen2P-rescue:LP5912-5.0-RoMeLa_Motor
- U7: symbol Motor_Gen2-rescue:ADS8353-RoMeLa_Motor -> Motor_Gen2P-rescue:ADS8353-RoMeLa_Motor
Connections:
- wire segments 81 -> 47
Other:
- note added: "Changed to direct drive \nfor space saving."
