File: pcb/split/gen2P/Power_Stage.sch (KiCad schematic (older format))
At the start: 41 parts, among them Q1 CSD88599Q5DC, Q2 CSD88599Q5DC, Q3 CSD88599Q5DC, U2 TLV76733DRVR, U3 DRV8320RS

Commit message: updated schematics and added split PCB.
Parts:
- removed C13, C14: 10uF 100v, Capacitor_SMD:C_2220_5650Metric, symbol Motor_Gen2-rescue:C_Small-Device
- removed C16: 104, Capacitor_SMD:C_0402_1005Metric, symbol Motor_Gen2-rescue:C_Small-Device
- removed C22, C23, C24: 4.7nF 100v, Capacitor_SMD:C_0402_1005Metric, symbol Motor_Gen2-rescue:C_Small-Device
- removed C8: 100uF, Capacitor_THT:CP_Radial_D10.0mm_P5.00mm, symbol Motor_Gen2-rescue:CP1_Small-Device
- removed Q1, Q2, Q3: CSD88599Q5DC, RoMeLa_Motor:TI_Q5DC, symbol Motor_Gen2-rescue:CSD88599Q5DC-RoMeLa_Motor
- removed R10, R11, R9: 2.21Ω, Resistor_SMD:R_0603_1608Metric, symbol Motor_Gen2-rescue:R_Small-Device
- added Q1, Q2, Q3, Q4, Q5, Q6: NMOS, RoMeLa_Motor:DFNW8_8.3x8.4_short, symbol Motor_Gen2P-rescue:Q_NMOS_GSD-Device
- C10, C11, C12, C9: value 10uF 100v -> 22uF 100v; symbol Motor_Gen2-rescue:C_Small-Device -> Motor_Gen2P-rescue:C_Small-Device
- C15: footprint Capacitor_SMD:C_2220_5650Metric -> Capacitor_SMD:C_1210_3225Metric; symbol Motor_Gen2-rescue:C_Small-Device -> Motor_Gen2P-rescue:C_Small-Device
- C17, C18, C19, C20, C21, C25, C28, C29, C30, C31, C32: symbol Motor_Gen2-rescue:C_Small-Device -> Motor_Gen2P-rescue:C_Small-Device
- C27: value 1uF 16v -> 2.2uF 16v; footprint Capacitor_SMD:C_0805_2012Metric -> Capacitor_SMD:C_0603_1608Metric; symbol Motor_Gen2-rescue:C_Small-Device -> Motor_Gen2P-rescue:C_Small-Device
- D4: symbol Motor_Gen2-rescue:D_Schottky_Small-Device -> Motor_Gen2P-rescue:D_Schottky_Small-Device
- L1: footprint Inductor_SMD:L_Taiyo-Yuden_MD-4040 -> RoMeLa_Motor:L_Taiyo-Yuden_DND4040WK; symbol Motor_Gen2-rescue:L_Small-Device -> Motor_Gen2P-rescue:L_Small-Device
- R12, R13: value R001 -> 500U; symbol Motor_Gen2-rescue:R_Shunt-Device -> Motor_Gen2P-rescue:R_Shunt-Device
- R14, R15, R6, R7: symbol Motor_Gen2-rescue:R_Small-Device -> Motor_Gen2P-rescue:R_Small-Device
- R8: footprint Resistor_SMD:R_0402_1005Metric -> NetTie:NetTie-2_SMD_Pad0.5mm; symbol Motor_Gen2-rescue:R_Small-Device -> Motor_Gen2P-rescue:R_Small-Device
- U2: symbol Motor_Gen2-rescue:TLV76733DRVR-RoMeLa_Motor -> Motor_Gen2P-rescue:TLV76733DRVR-RoMeLa_Motor
- U3: symbol Motor_Gen2-rescue:DRV8320RS-RoMeLa_Motor -> Motor_Gen2P-rescue:DRV8320RS-RoMeLa_Motor
Connections:
- wire segments 137 -> 130
